Commit message: New update with nav2 and twist_launch

File: description/camera.xacro (robot description, xacro)
@@ -24,5 +24,5 @@
         <sensor name="camera" type="camera">
             <pose> 0 0 0 0 0 0 </pose>
-            <visualize>true</visualize>
+            <visualize>false</visualize>
             <update_rate>10</update_rate>
             <camera>

File: description/gazebo_control.xacro (robot description, xacro)
@@ -6,5 +6,5 @@
             <left_joint>left_wheel_joint</left_joint>
             <right_joint>right_wheel_joint</right_joint>
-            <wheel_separation>0.56</wheel_separation>
+            <wheel_separation>0.44</wheel_separation>
             <wheel_diameter>0.2</wheel_diameter>
             <!-- Limits -->

File: description/lidar.xacro (robot description, xacro)
@@ -1,4 +1,20 @@
 <?xml version="1.0"?>
 <robot xmlns:xacro="http://www.ros.org/wiki/xacro" >
+    <link name="laser_frame">
+        <visual>
+            <geometry>
+                <cylinder radius="0.05" length="0.04"/>
+            </geometry>
+            <material name="black"/>
+        </visual>
+        <collision>
+            <geometry>
+                <cylinder radius="0.05" length="0.04"/>
+            </geometry>
+        </collision>
+        <xacro:inertial_cylinder mass="0.1" length="0.04" radius="0.05">
+            <origin xyz="0.07 0 0.329" rpy="0 0 0"/>
+        </xacro:inertial_cylinder>
+    </link>
     <joint name="laser_joint" type="fixed">
         <parent link="chassis"/>
@@ -6,47 +22,32 @@
         <origin xyz="0.07 0 0.329" rpy="0 0 0"/>
     </joint>
-    <link name="laser_frame">
-    <visual>
-        <geometry>
-            <cylinder radius="0.05" length="0.04"/>
-        </geometry>
-        <material name="black"/>
-    </visual>
-    <collision>
-        <geometry>
-            <cylinder radius="0.05" length="0.04"/>
-        </geometry>
-    </collision>
-    <xacro:inertial_cylinder mass="0.1" length="0.04" radius="0.05">
-        <origin xyz="0 0 0" rpy="0 0 0"/>
-    </xacro:inertial_cylinder>
-</link>
-<gazebo reference="laser_frame">
-    <material>Gazebo/Black</material>
-    <sensor name="laser" type="ray">
-        <pose> 0 0 0 0 0 0 </pose>
-        <visualize>true</visualize>
-        <update_rate>10</update_rate>
-        <ray>
-            <scan>
-                <horizontal>
-                    <samples>360</samples>
-                    <min_angle>-3.14</min_angle>
-                    <max_angle>3.14</max_angle>
-                </horizontal>
-            </scan>
-            <range>
-                <min>0.1</min>
-                <max>15</max>
-            </range>
-        </ray>
-        <plugin name="laser_controller" filename="libgazebo_ros_ray_sensor.so">
-            <ros>
-                <argument>~/out:=scan</argument>
-            </ros>
-            <output_type>sensor_msgs/LaserScan</output_type>
-            <frame_name>laser_frame</frame_name>
-        </plugin>
-    </sensor>
-</gazebo>
+    <gazebo reference="laser_frame">
+        <material>Gazebo/Black</material>
+        <sensor name="laser" type="ray">
+            <visualize>true</visualize>
+            <update_rate>10</update_rate>
+            <ray>
+                <scan>
+                    <horizontal>
+                        <samples>360</samples>
+                        <resolution>1.000000</resolution>
+                        <min_angle>-3.14</min_angle>
+                        <max_angle>3.14</max_angle>
+                    </horizontal>
+                </scan>
+                <range>
+                    <min>0.1</min>
+                    <max>15</max>
+                    <resolution>0.015000</resolution>
+                </range>
+            </ray>
+            <plugin name="laser_controller" filename="libgazebo_ros_ray_sensor.so">
+                <ros>
+                    <argument>~/out:=scan</argument>
+                </ros>
+                <output_type>sensor_msgs/LaserScan</output_type>
+                <frame_name>laser_frame</frame_name>
+            </plugin>
+        </sensor>
+    </gazebo>
 </robot>

File: description/robot_core.xacro (robot description, xacro)
@@ -27,10 +27,10 @@
         <parent link="base_link"/>
         <child link="base_footprint"/>
-        <origin xyz="0 0 0" rpy="0 0 0"/>
+        <origin xyz="0 0 0.1" rpy="0 0 0"/>
     </joint>
     <link name="base_footprint"></link>
     <!-- CHASSIS LINK -->
     <joint name="chassis_joint" type="fixed">
-        <parent link="base_link"/>
+        <parent link="base_footprint"/>
         <child link="chassis"/>
         <origin xyz="-0.1 0 0"/>
@@ -44,13 +44,17 @@
             <material name="yellow"/>
         </visual>
-        <collision>
+        <!-- <collision>
             <origin xyz="0.426 0 0.130"/>
             <geometry>
-                <box size="0.001 0.001 0.001"/>
+                <box size="0.01 0.01 0.01"/>
+                <box size="0.810 0.500 0.259"/>
             </geometry>
-        </collision>
-        <xacro:inertial_box mass="1" x="0.810" y="0.500" z="0.259">
+        </collision> -->
+        <xacro:inertial_box mass="0.3" x="0.810" y="0.500" z="0.259">
             <origin xyz="0.426 0 0.130" rpy="0 0 0"/>
         </xacro:inertial_box>
+        <!-- <xacro:inertial_box mass="1" x="0.810" y="0.500" z="0.259">
+            <origin xyz="0 0 0" rpy="0 0 0"/>
+        </xacro:inertial_box> -->
     </link>
     <gazebo reference="chassis">
@@ -59,5 +63,5 @@
     <!-- LEFT WHEEL LINK -->
     <joint name="left_wheel_joint" type="continuous">
-        <parent link="base_link"/>
+        <parent link="base_footprint"/>
         <child link="left_wheel"/>
         <origin xyz="0 0.220 0" rpy="-${pi/2} 0 0" />
@@ -85,5 +89,5 @@
     <!-- RIGHT WHEEL LINK -->
     <joint name="right_wheel_joint" type="continuous">
-        <parent link="base_link"/>
+        <parent link="base_footprint"/>
         <child link="right_wheel"/>
         <origin xyz="0 -0.220 0" rpy="${pi/2} 0 0" />
@@ -127,6 +131,6 @@
             </geometry>
         </collision>
-        <xacro:inertial_sphere mass="0.1" radius="0.0675">
-            <origin xyz="0 0 0" rpy="0 0 0"/>
+        <xacro:inertial_sphere mass="0.3" radius="0.0675">
+            <origin xyz="0 0 0"/>
         </xacro:inertial_sphere>
     </link>
